File: RaspberryMesh.brd (EAGLE design)
At the start: 85.1 x 55.9 mm, 77 parts, among them IC1 MPL115A, IC2 DS1307, IC3 TEMT6000, IC4 MC34063, IC5 ATmega128RFA1, J10 ISP, J2 12V Supply, J3 RASPBERRY-PI, Q1 32768 Hz, Q2 2N7002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

Commit message: foo
Connections:
- removed net N$15: LED3.C, R5.1
- new net N$8: LED3.A, R5.1
- net GND: now also LED3.C; no longer LED3.A
