File: RaspberryMesh.sch (EAGLE design)
At the start: 77 parts, among them IC1 MPL115A, IC2 DS1307, IC3 TEMT6000, IC4 MC34063, IC5 ATmega128RFA1, J10 ISP, J2 12V Supply, J3 RASPBERRY-PI, Q1 32768 Hz, Q2 2N7002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

Commit message: foo
Connections:
- removed net N$15: LED3.C, R5.1
- new net N$8: LED3.A, R5.1
- net GND: now also LED3.C; no longer LED3.A
Changed lines of the file:
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@@
 <text x="45.72" y="198.12" size="2.1844" layer="97">http://ohwr.org/cernohl</text>
 <wire x1="215.9" y1="264.16" x2="215.9" y2="220.98" width="0.1524" layer="98" style="shortdash"/>
-<text x="25.4" y="154.94" size="1.778" layer="97" ratio="16">ISP programmer must only supply 3.3V power and logic.</text>
+<text x="25.4" y="154.94" size="1.778" layer="97">ISP programmer must only supply 3.3V power and logic.</text>
 <wire x1="241.3" y1="30.48" x2="17.78" y2="30.48" width="0.1524" layer="98" style="shortdash"/>
 <wire x1="17.78" y1="167.64" x2="17.78" y2="30.48" width="0.1524" layer="98" style="shortdash"/>
@@
 <instance part="U$42" gate="G$1" x="238.76" y="281.94"/>
 <instance part="U$43" gate="G$1" x="198.12" y="281.94"/>
-<instance part="LED3" gate="G$1" x="205.74" y="289.56" smashed="yes" rot="R90">
-<attribute name="NAME" x="203.2" y="284.48" size="1.016" layer="95"/>
-<attribute name="VALUE" x="203.2" y="281.94" size="1.016" layer="96"/>
-<attribute name="PACKAGE" x="203.2" y="279.4" size="1.016" layer="96"/>
+<instance part="LED3" gate="G$1" x="208.28" y="289.56" smashed="yes" rot="MR90">
+<attribute name="NAME" x="200.66" y="284.48" size="1.016" layer="95"/>
+<attribute name="VALUE" x="205.74" y="284.48" size="1.016" layer="96"/>
+<attribute name="PACKAGE" x="205.74" y="281.94" size="1.016" layer="96"/>
 </instance>
 <instance part="LED2" gate="G$1" x="238.76" y="304.8" smashed="yes" rot="R270">
@@
 <segment>
 <pinref part="U$43" gate="G$1" pin="GND"/>
-<wire x1="198.12" y1="284.48" x2="198.12" y2="289.56" width="0.1524" layer="91"/>
-<wire x1="198.12" y1="289.56" x2="203.2" y2="289.56" width="0.1524" layer="91"/>
 <pinref part="IC2" gate="G$1" pin="GND"/>
 <wire x1="200.66" y1="297.18" x2="198.12" y2="297.18" width="0.1524" layer="91"/>
 <wire x1="198.12" y1="297.18" x2="198.12" y2="289.56" width="0.1524" layer="91"/>
+<pinref part="LED3" gate="G$1" pin="C"/>
+<wire x1="198.12" y1="289.56" x2="198.12" y2="284.48" width="0.1524" layer="91"/>
+<wire x1="203.2" y1="289.56" x2="198.12" y2="289.56" width="0.1524" layer="91"/>
 <junction x="198.12" y="289.56"/>
-<pinref part="LED3" gate="G$1" pin="A"/>
 </segment>
 </net>
@@
 </segment>
 </net>
-<net name="N$15" class="0">
-<segment>
-<pinref part="R5" gate="G$1" pin="1"/>
-<wire x1="210.82" y1="289.56" x2="213.36" y2="289.56" width="0.1524" layer="91"/>
-<pinref part="LED3" gate="G$1" pin="C"/>
-</segment>
-</net>
 <net name="N$16" class="0">
 <segment>
@@
 </segment>
 </net>
+<net name="N$8" class="0">
+<segment>
+<pinref part="LED3" gate="G$1" pin="A"/>
+<pinref part="R5" gate="G$1" pin="1"/>
+<wire x1="210.82" y1="289.56" x2="213.36" y2="289.56" width="0.1524" layer="91"/>
+</segment>
+</net>
